File: PulseWristTrack.kicad_pcb (KiCad board)
At the start: 4 copper layers, 36 x 36 mm, 18 parts, among them J1 LiPo, Q1 BSS138, Q2 BSS138, SW1 JS202011MQN, U1 XIAO nRF52840 Sense, U2 MAX30102, U3 AP2112K-1.8

Commit message: auto-backup 2026-07-24 19:26:27
Parts:
- J1: value LiPo -> BATT_JST_PH
- SW1: value JS202011MQN -> JS102011SAQN; footprint Button_Switch_SMD:SW_SPDT_PCM12 -> Button_Switch_SMD:SW_SPDT_CK_JS102011SAQN
- U1: value XIAO nRF52840 Sense -> XIAO_nRF52840_Sense
- moved J1 88.2 mm to (-8.00, -12.4)
- moved SW1 85.0 mm to (8.00, -10.0)
- moved C2 84.3 mm to (-2.50, -8.00)
- moved Q1 80.3 mm to (-6.00, 3.00)
- moved C3 79.9 mm to (2.00, -7.00), turned to 0 degrees
- moved U3 76.5 mm to (-5.00, -5.00)
- moved C1 72.8 mm to (-9.00, -2.00)
- moved MH1 70.7 mm to (-12.0, 0.00)
- moved MH2 70.7 mm to (12.0, 0.00)
- moved U2 70.7 mm to (0.00, 0.00)
- moved R5 70.5 mm to (0.00, 9.50)
- moved U1 66.6 mm to (0.00, 3.00)
- moved Q2 65.9 mm to (6.00, 3.00)
- moved R4 63.2 mm to (6.00, 8.00), turned to 0 degrees
- moved R1 62.8 mm to (-6.00, 8.00), turned to 0 degrees
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Connections:
- J1 pad 1: BAT_RAW -> BAT+
- SW1 pad 1: BAT_RAW -> BAT_SW
- SW1 pad 2: BAT_SW -> BAT+
- U2 pad 1: (no net) -> SCL_1V8
- U2 pad 11: +1V8 -> GND
- U2 pad 12: GND -> INT
- U2 pad 2: SCL_1V8 -> SDA_1V8
- U2 pad 3: SDA_1V8 -> GND
- U2 pad 5: (no net) -> +3V3
- U2 pad 6: (no net) -> +3V3
- U2 pad 9: +3V3 -> +1V8
Routing:
- net BAT+: track 0.00 -> 25.8 mm
- net SCL_3V3: track 34.5 -> 12.6 mm
- net BAT_RAW: track 14.1 -> 0.00 mm
- net SDA_3V3: track 16.1 -> 28.3 mm, vias 2 -> 1
- net BAT_SW: track 20.2 -> 31.8 mm
- net +1V8: track 51.3 -> 44.5 mm
- net SCL_1V8: track 12.3 -> 16.6 mm
- net SDA_1V8: track 25.4 -> 21.4 mm
- net +3V3: track 2.28 -> 0.40 mm, vias 0 -> 9
- net GND: track 0.00 -> 0.40 mm, vias 0 -> 8
- net INT: track 19.6 -> 19.7 mm, vias 1 -> 2

Commit message: auto-backup 2026-07-24 20:26:27
Parts:
- moved J1 4.40 mm to (-8.00, -8.00)
- moved SW1 2.00 mm to (8.00, -8.00)
Routing:
- net BAT+: track 25.8 -> 19.4 mm
- net BAT_SW: track 31.8 -> 29.8 mm
- net GND: vias 8 -> 9
- net +3V3: vias 9 -> 10
Changed lines of the file:
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@@
 	(footprint "Connector_JST:JST_PH_S2B-PH-K_1x02_P2.00mm_Horizontal"
 		(layer "F.Cu")
-		(at -8 -12.4)
+		(at -8 -8)
 		(descr "JST PH series connector, S2B-PH-K (http://www.jst-mfg.com/product/pdf/eng/ePH.pdf)")
 		(tags "connector JST PH horizontal")
@@
 		(fp_rect
 			(start -2.45 -1.85)
-			(end 4.45 6.75)
+			(end 4.45 2.3)
 			(stroke
 				(width 0.05)
@@
 	(footprint "Button_Switch_SMD:SW_SPDT_CK_JS102011SAQN"
 		(layer "F.Cu")
-		(at 8 -10)
+		(at 8 -8)
 		(descr "Sub-miniature slide switch, right-angle, http://www.ckswitches.com/media/1422/js.pdf")
 		(tags "switch spdt")
@@
 		(fp_line
 			(start -3.25 2.25)
-			(end -3.25 2.75)
+			(end -2.5 2.25)
 			(stroke
 				(width 0.05)
@@
 		)
 		(fp_line
-			(start -3.25 2.75)
-			(end -2.5 2.75)
+			(start -2.5 2.25)
+			(end 2.5 2.25)
 			(stroke
 				(width 0.05)
@@
 		)
 		(fp_line
-			(start -2.5 2.75)
-			(end -2.5 4.25)
-			(stroke
-				(width 0.05)
-				(type solid)
-			)
-			(layer "F.CrtYd")
-		)
-		(fp_line
-			(start -2.5 4.25)
-			(end 2.5 4.25)
-			(stroke
-				(width 0.05)
-				(type solid)
-			)
-			(layer "F.CrtYd")
-		)
-		(fp_line
-			(start 2.5 2.5)
-			(end 3.25 2.5)
-			(stroke
-				(width 0.05)
-				(type solid)
-			)
-			(layer "F.CrtYd")
-		)
-		(fp_line
-			(start 2.5 4.25)
-			(end 2.5 2.5)
+			(start 2.5 2.25)
+			(end 3.25 2.25)
 			(stroke
 				(width 0.05)
@@
 		)
 		(fp_line
-			(start 3.25 2.5)
-			(end 3.25 2.25)
-			(stroke
-				(width 0.05)
-				(type solid)
-			)
-			(layer "F.CrtYd")
-		)
-		(fp_line
 			(start 3.5 -4.5)
 			(end -3.5 -4.5)
@@
 	)
 	(segment
-		(start -8 -12.4)
-		(end -8 -8)
-		(width 0.4)
-		(layer "F.Cu")
-		(net "BAT+")
-	)
-	(segment
-		(start 8 -12.75)
-		(end 8 -10.75)
-		(width 0.4)
-		(layer "F.Cu")
-		(net "BAT+")
-	)
-	(segment
 		(start -4.9972 -6.5938)
 		(end -6.5938 -6.5938)
@@
 	)
 	(via
+		(at -0.1 1)
+		(size 0.4)
+		(drill 0.2)
+		(layers "F.Cu" "B.Cu")
+		(net "GND")
+	)
+	(via
 		(at -9 -2.95)
 		(size 0.6)
@@
 	)
 	(segment
-		(start 5.5 -12.75)
-		(end 5.5 -10.75)
-		(width 0.4)
-		(layer "F.Cu")
-		(net "BAT_SW")
-	)
-	(segment
 		(start -9.8046 -8.2793)
 		(end -9.8046 2.0854)
@@
 		(size 0.6)
 		(drill 0.3)
+		(layers "F.Cu" "B.Cu")
+		(net "+3V3")
+	)
+	(via
+		(at -0.8 0.8)
+		(size 0.6)
+		(drill 0.3)
